File: 0039_Force_Module_Classic.kicad_sch (KiCad schematic)
At the start: 7 parts, among them J1 Force Sensor, U1 TLV521DCKR

Commit message: Add files via upload
Parts:
- added D1: LED, LED_SMD:LED_0805_2012Metric, symbol Device:LED
- added R3: R, Resistor_SMD:R_0805_2012Metric, symbol Device:R
- added U2: ~, Moduler_:pin_header, symbol moduler_pin:air
- C1, C2, C3: footprint (none) -> Capacitor_SMD:C_0805_2012Metric
- J1: footprint (none) -> TerminalBlock_Phoenix:TerminalBlock_Phoenix_MPT-0,5-2-2.54_1x02_P2.54mm_Horizontal
- R1, R2: footprint (none) -> Resistor_SMD:R_0805_2012Metric
- U1: footprint SOT65P210X110-5N -> meminle:SOT65P210X110-5N
Connections:
- net +3V3: now also R3.1, U2.8
- net GND: now also D1.1 (K), U2.9
- net OUT: now also U2.12
- new net: D1.2 (A), R3.2
- no-connect marks 0 -> 15
Other:
- note added: "AIR PIN"
- note added: "SENSOR"
- moved on the sheet: C1, C2, C3, J1, R1, R2, U1
